Commit message: my_robot rev02 created

File: my_robot_superseded/my_robot_rev01/urdf/my_robot.urdf (robot description, URDF)
Before this commit: robot my_robot, 5 links, 4 joints
Links:
- link base_link: mass 3.1224 -> 3.12236517080469
Joints:
- joint left_front_wheel_joint: origin xyz=0.256 0.22035 -0.1953 rpy=-1.5708 1.2311 -3.1416 -> xyz=0.2775 -0.256 -0.1953 rpy=1.5708 -0.83796 -1.5708
- joint left_rear_wheel_joint: origin xyz=-0.256 0.22035 -0.1953 rpy=-1.5708 -0.33051 3.1416 -> xyz=0.2775 0.256 -0.1953 rpy=1.5708 0.72361 -1.5708
- joint right_front_wheel_joint: origin xyz=0.256 -0.22035 -0.1953 rpy=1.5708 -1.4489 3.1416 -> xyz=-0.2775 -0.256 -0.1953 rpy=1.5708 1.2996 1.5708
- joint right_rear_wheel_joint: origin xyz=-0.256 -0.22035 -0.1953 rpy=1.5708 1.2718 -3.1416 -> xyz=-0.2775 0.256 -0.1953 rpy=-1.5708 -0.87872 -1.5708
