Commit message: my_robot rev01 created

File: my_robot/urdf/my_robot.urdf (robot description, URDF)
Before this commit: robot my_robot, 5 links, 4 joints
Links:
- removed link left_back_wheel
- removed link right_back_wheel
- added link left_rear_wheel, mass 8.232; collision mesh filename=package://my_robot/meshes/left_rear_wheel.STL; visual mesh filename=package://my_robot/meshes/left_rear_wheel.STL
- added link right_rear_wheel, mass 8.232; collision mesh filename=package://my_robot/meshes/right_rear_wheel.STL; visual mesh filename=package://my_robot/meshes/right_rear_wheel.STL
- link base_link: mass 3.12236517080471 -> 3.12236517080469
Joints:
- removed joint left_back_wheel_joint
- removed joint right_back_wheel_joint
- added joint left_rear_wheel_joint: type continuous, parent base_link, child left_rear_wheel, origin xyz=0.2775 0.256 -0.1953 rpy=1.5708 0.72361 -1.5708, axis 0 0 1
- added joint right_rear_wheel_joint: type continuous, parent base_link, child right_rear_wheel, origin xyz=-0.2775 0.256 -0.1953 rpy=-1.5708 -0.87872 -1.5708, axis 0 0 1
- joint left_front_wheel_joint: origin xyz=0.2446 0.1953 0.22035 rpy=3.1416 0 0.34104 -> xyz=0.2775 -0.256 -0.1953 rpy=1.5708 -0.83796 -1.5708
- joint right_front_wheel_joint: origin xyz=0.2446 0.1953 -0.22035 rpy=0 0 2.5629 -> xyz=-0.2775 -0.256 -0.1953 rpy=1.5708 1.2996 1.5708

File: my_robot_superseded/my_robot/urdf/my_robot.urdf (robot description, URDF)
Before this commit: robot my_robot, 5 links, 4 joints
Links:
- removed link left_rear_wheel
- removed link right_rear_wheel
- added link left_back_wheel, mass 8.232; collision mesh filename=package://my_robot/meshes/left_back_wheel.STL; visual mesh filename=package://my_robot/meshes/left_back_wheel.STL
- added link right_back_wheel, mass 8.232; collision mesh filename=package://my_robot/meshes/right_back_wheel.STL; visual mesh filename=package://my_robot/meshes/right_back_wheel.STL
- link base_link: mass 3.12236517080469 -> 3.12236517080471
Joints:
- removed joint left_rear_wheel_joint
- removed joint right_rear_wheel_joint
- added joint left_back_wheel_joint: type continuous, parent base_link, child left_back_wheel, origin xyz=-0.2674 0.1953 0.22035 rpy=-3.1416 0 1.9026, axis 0 0 1
- added joint right_back_wheel_joint: type continuous, parent base_link, child right_back_wheel, origin xyz=-0.2674 0.1953 -0.22035 rpy=0 0 -1.436, axis 0 0 1
- joint left_front_wheel_joint: origin xyz=0.2775 -0.256 -0.1953 rpy=1.5708 -0.83796 -1.5708 -> xyz=0.2446 0.1953 0.22035 rpy=3.1416 0 0.34104
- joint right_front_wheel_joint: origin xyz=-0.2775 -0.256 -0.1953 rpy=1.5708 1.2996 1.5708 -> xyz=0.2446 0.1953 -0.22035 rpy=0 0 2.5629

Commit message: my_robot rev02 created

File: my_robot/urdf/my_robot.urdf (robot description, URDF)
Before this commit: robot my_robot, 5 links, 4 joints
Links:
- link base_link: mass 3.1224 -> 3.12236517080468
- link left_front_wheel: mass 8.232 -> 8.23195517435844
- link left_rear_wheel: mass 8.232 -> 8.23195517435845
- link right_front_wheel: mass 8.232 -> 8.2319551743634
- link right_rear_wheel: mass 8.232 -> 8.23195748178054
Joints:
- joint right_front_wheel_joint: origin xyz=0.256 -0.22035 -0.1953 rpy=1.5708 -1.4489 3.1416 -> xyz=0.256 -0.33465 -0.1953 rpy=1.5708 -1.4489 3.1416
