Commit message: my_robot collision mesh files added

File: my_robot_collision/urdf/my_robot_collision.urdf (robot description, URDF)
Before this commit: robot my_robot, 5 links, 4 joints
Links:
- link base_link: mass 3.12236517080468 -> 3.1224; geometry collision mesh filename=package://my_robot_collision/meshes/base_link.STL; visual mesh filename=package://my_robot_collision/meshes/base_link.STL
- link left_front_wheel: mass 8.23195517435844 -> 9.1523; geometry collision mesh filename=package://my_robot_collision/meshes/left_front_wheel.STL; visual mesh filename=package://my_robot_collision/meshes/left_front_wheel.STL
- link left_rear_wheel: mass 8.23195517435845 -> 9.1523; geometry collision mesh filename=package://my_robot_collision/meshes/left_rear_wheel.STL; visual mesh filename=package://my_robot_collision/meshes/left_rear_wheel.STL
- link right_front_wheel: mass 8.2319551743634 -> 9.1523; geometry collision mesh filename=package://my_robot_collision/meshes/right_front_wheel.STL; visual mesh filename=package://my_robot_collision/meshes/right_front_wheel.STL
- link right_rear_wheel: mass 8.23195748178054 -> 9.1523; geometry collision mesh filename=package://my_robot_collision/meshes/right_rear_wheel.STL; visual mesh filename=package://my_robot_collision/meshes/right_rear_wheel.STL
